File: PCB/clock.kicad_pcb (KiCad board)
At the start: 2 copper layers, 210 x 105 mm, 112 parts, among them J1 PWR, J2 PWR, J3 EXT_TEMP, J4 EXT_TEMP, J5 PROG, Q1 BSS138, Q2 BSS138, Q3 BSS138, SW1 ENTER, SW2 PLUS, SW3 MINUS, SW4 ESC, U1 D148K, U10 DS9503P1, U11 D148K, U12 D148K, U13 D148K, U14 D148K, U15 D148K, U16 D148K, U17 D148K, U18 D148K, U19 MAX7219, U2 D148K, U20 DS3231MZ, U21 DS3231M, U22 D148K, U23 D148K, U24 D148K, U25 D148K, U26 D148K, U27 D148K, U28 MAX7219, U29 STM32F030F4Px, U3 D148K, U4 D148K, U5 D148K, U6 D148K, U7 LM1117DT-3.3, U8 MAX7219, U9 DS2482, Y1 10MHz

Commit message: PCB updated with final component values
Parts:
- D6: value MRA4007 -> SS16 SHOTTKY
- R1, R2, R3, R4: value 100 -> 0
- R13, R18: value 10k -> 47k
- R20, R21: value 3k3 -> 2k2
- R5: value 10k -> 13k7
- Y1: value 10MHz -> 8MHz

Commit message: Logic shifter resistors readjustment
Parts:
- R10, R6, R8: value 10k -> 2k2
Changed lines of the file:
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@@
 			)
 		)
-		(property "Value" "10k"
+		(property "Value" "2k2"
 			(at 0 -1.82 0)
 			(layer "B.Fab")
@@
 		(fp_arc
 			(start 21.59 0.25)
-			(mid 21.329578 0.950494)
+			(mid 21.329583 0.950487)
 			(end 20.68 1.32)
 			(stroke
@@
 		(fp_arc
 			(start 20.68 -1.32)
-			(mid 21.329593 -0.950487)
+			(mid 21.329556 -0.950479)
 			(end 21.59 -0.25)
 			(stroke
@@
 			)
 		)
-		(property "Value" "10k"
+		(property "Value" "2k2"
 			(at 2.375 -1.82 0)
 			(layer "B.Fab")
@@
 			)
 		)
-		(property "Value" "10k"
+		(property "Value" "2k2"
 			(at 0 -1.82 0)
 			(layer "B.Fab")
